Commit message: new moveit_config version

File: erl2/urdf/m2wr_arm2.xacro (robot description, xacro)
@@ -263,5 +263,5 @@
   	</visual>
   </link>
-    <joint name="cluedo_link_joint" type="revolute">
+    <joint name="cluedo_joint" type="revolute">
   	<axis xyz="1 0 0"/>
   	<limit effort="1000.0" lower="-1.8" upper="1.8" velocity="0.5"/>
@@ -364,4 +364,14 @@
 	</actuator>
 </transmission>
+<transmission name="cluedo_joint_trans">
+	<type>transmission_interface/SimpleTransmission</type>
+	<joint name="cluedo_joint">
+		<hardwareInterface>hardware_interface/EffortJointInterface</hardwareInterface>
+	</joint>
+	<actuator name="motor5">
+		<hardwareInterface>hardware_interface/EffortJointInterface</hardwareInterface>
+		<mechanicalInterface>1</mechanicalInterface>
+	</actuator>
+</transmission>
 <transmission name="left_grip_trans">
 	<type>transmission_interface/SimpleTransmission</type>
@@ -369,5 +379,5 @@
 		<hardwareInterface>hardware_interface/EffortJointInterface</hardwareInterface>
 	</joint>
-	<actuator name="motor5">
+	<actuator name="motor6">
 		<hardwareInterface>hardware_interface/EffortJointInterface</hardwareInterface>
 		<mechanicalInterface>1</mechanicalInterface>
@@ -379,5 +389,5 @@
 		<hardwareInterface>hardware_interface/EffortJointInterface</hardwareInterface>
 	</joint>
-	<actuator name="motor6">
+	<actuator name="motor7">
 		<hardwareInterface>hardware_interface/EffortJointInterface</hardwareInterface>
 		<mechanicalInterface>1</mechanicalInterface>

File: erl2/urdf/robot.urdf (robot description, URDF)
Before this commit: robot m2wr, 12 links, 11 joints
Joints:
- removed joint cluedo_link_joint
- added joint cluedo_joint: type revolute, parent arm_link_04, child cluedo_link, origin xyz=0 0 0 rpy=0 0 0, axis 1 0 0, limit lower=-1.8 upper=1.8 effort=1000.0 velocity=0.5

Commit message: new moveit version, add init arm position

File: erl2/urdf/m2wr_arm2.xacro (robot description, xacro)
@@ -140,4 +140,31 @@
   	<child link="arm_base_link"/>
   </joint>
+  <link name="arm_link_0">
+  	<inertial>
+  		<mass value="0.025"/>
+  		<origin xyz="0 0 0" rpy="0 0 0" />
+  		<inertia ixx="0.000010279" ixy="0" ixz="0" iyy="0.000010279" iyz="0" izz="0.000007225"/>
+  	</inertial>
+  	<collision>
+  	  <origin xyz="0 0 ${len_coeff*0}" rpy="0 0 0"/>
+      <geometry>
+        <cylinder radius="0.04" length="${len_coeff*0}"/>
+      </geometry>
+  	</collision>
+  	<visual>
+  	  <origin xyz="0 0 ${len_coeff*0}" rpy="0 0 0"/>
+      <geometry>
+        <cylinder radius="0.04" length="${len_coeff*0}"/>
+      </geometry>
+      <material name="red" />
+  	</visual>
+  </link>
+  <joint name="arm_joint_0" type="revolute">
+  	<axis xyz="0 1 0"/>
+  	<limit effort="1000.0" lower="-1.7" upper="1.7" velocity="0.2"/>
+  	<origin rpy="0 0 0" xyz="0 0 ${len_coeff*0.0001}"/>
+  	<parent link="arm_base_link"/>
+  	<child link="arm_link_0"/>
+  </joint>
   <link name="arm_link_01">
   	<inertial>
@@ -164,5 +191,5 @@
   	<limit effort="1000.0" lower="-3.14" upper="3.14" velocity="0.2"/>
   	<origin rpy="0 0 0" xyz="0 0 ${len_coeff*0.5}"/>
-  	<parent link="arm_base_link"/>
+  	<parent link="arm_link_0"/>
   	<child link="arm_link_01"/>
   </joint>
@@ -324,4 +351,14 @@
   	<child link="left_grip_link"/>
   </joint>
+<transmission name="arm_joint_0_trans">
+	<type>transmission_interface/SimpleTransmission</type>
+	<joint name="arm_joint_0">
+		<hardwareInterface>hardware_interface/EffortJointInterface</hardwareInterface>
+	</joint>
+	<actuator name="motor0">
+		<hardwareInterface>hardware_interface/EffortJointInterface</hardwareInterface>
+		<mechanicalInterface>1</mechanicalInterface>
+	</actuator>
+</transmission>
 <transmission name="arm_joint_01_trans">
 	<type>transmission_interface/SimpleTransmission</type>

File: erl2/urdf/robot.urdf (robot description, URDF)
Before this commit: robot m2wr, 12 links, 11 joints
Links:
- added link arm_link_0, mass 0.025; collision cylinder length=0.0 radius=0.04; visual cylinder length=0.0 radius=0.04
Joints:
- added joint arm_joint_0: type revolute, parent arm_base_link, child arm_link_0, origin xyz=0 0 8e-05 rpy=0 0 0, axis 0 1 0, limit lower=-1.7 upper=1.7 effort=1000.0 velocity=0.2
- joint arm_joint_01: parent arm_base_link -> arm_link_0

Commit message: trials

File: erl2/urdf/m2wr_arm2.xacro (robot description, xacro)
@@ -140,31 +140,4 @@
   	<child link="arm_base_link"/>
   </joint>
-  <link name="arm_link_0">
-  	<inertial>
-  		<mass value="0.025"/>
-  		<origin xyz="0 0 0" rpy="0 0 0" />
-  		<inertia ixx="0.000010279" ixy="0" ixz="0" iyy="0.000010279" iyz="0" izz="0.000007225"/>
-  	</inertial>
-  	<collision>
-  	  <origin xyz="0 0 ${len_coeff*0}" rpy="0 0 0"/>
-      <geometry>
-        <cylinder radius="0.04" length="${len_coeff*0}"/>
-      </geometry>
-  	</collision>
-  	<visual>
-  	  <origin xyz="0 0 ${len_coeff*0}" rpy="0 0 0"/>
-      <geometry>
-        <cylinder radius="0.04" length="${len_coeff*0}"/>
-      </geometry>
-      <material name="red" />
-  	</visual>
-  </link>
-  <joint name="arm_joint_0" type="revolute">
-  	<axis xyz="0 1 0"/>
-  	<limit effort="1000.0" lower="-1.7" upper="1.7" velocity="0.2"/>
-  	<origin rpy="0 0 0" xyz="0 0 ${len_coeff*0.0001}"/>
-  	<parent link="arm_base_link"/>
-  	<child link="arm_link_0"/>
-  </joint>
   <link name="arm_link_01">
   	<inertial>
@@ -191,5 +164,5 @@
   	<limit effort="1000.0" lower="-3.14" upper="3.14" velocity="0.2"/>
   	<origin rpy="0 0 0" xyz="0 0 ${len_coeff*0.5}"/>
-  	<parent link="arm_link_0"/>
+  	<parent link="arm_base_link"/>
   	<child link="arm_link_01"/>
   </joint>
@@ -351,14 +324,4 @@
   	<child link="left_grip_link"/>
   </joint>
-<transmission name="arm_joint_0_trans">
-	<type>transmission_interface/SimpleTransmission</type>
-	<joint name="arm_joint_0">
-		<hardwareInterface>hardware_interface/EffortJointInterface</hardwareInterface>
-	</joint>
-	<actuator name="motor0">
-		<hardwareInterface>hardware_interface/EffortJointInterface</hardwareInterface>
-		<mechanicalInterface>1</mechanicalInterface>
-	</actuator>
-</transmission>
 <transmission name="arm_joint_01_trans">
 	<type>transmission_interface/SimpleTransmission</type>

File: erl2/urdf/robot.urdf (robot description, URDF)
Before this commit: robot m2wr, 13 links, 12 joints
Links:
- removed link arm_link_0
Joints:
- removed joint arm_joint_0
- joint arm_joint_01: parent arm_link_0 -> arm_base_link

Commit message: bug to fix in launchng simulation, created launch files and correct CMakeList

File: erl2/urdf/m2wr_arm2.xacro (robot description, xacro)
@@ -189,5 +189,5 @@
   <joint name="arm_joint_02" type="revolute">
   	<axis xyz="1 0 0"/>
-  	<limit effort="1000.0" lower="-1.7" upper="-0.19" velocity="0.2"/>
+  	<limit effort="1000.0" lower="-3.14" upper="3.14" velocity="0.2"/>
   	<origin rpy="0 0 0" xyz="0 0 ${len_coeff*0.5}"/>
   	<parent link="arm_link_01"/>
@@ -216,5 +216,5 @@
   <joint name="arm_joint_03" type="revolute">
   	<axis xyz="1 0 0"/>
-  	<limit effort="1000.0" lower="-1.8" upper="-0.28" velocity="0.2"/>
+  	<limit effort="1000.0" lower="-3.14" upper="3.14" velocity="0.2"/>
   	<origin rpy="0 0 0" xyz="0 0 ${len_coeff}"/>
   	<parent link="arm_link_02"/>
@@ -264,5 +264,5 @@
   </link>
     <joint name="cluedo_joint" type="revolute">
-  	<axis xyz="1 0 0"/>
+  	<axis xyz="0 0 0"/>
   	<limit effort="1000.0" lower="-1.8" upper="1.8" velocity="0.5"/>
   	<origin rpy="0 0 0" xyz="0 0 0"/>
@@ -270,4 +270,32 @@
   	<child link="cluedo_link"/>
   </joint>
+  <link name="camera_link">
+	    <collision>
+	      <origin xyz="0 0 0.025" rpy="0 0 0"/>
+	      <geometry>
+		<box size="0.05 0.05 0.05"/>
+	      </geometry>
+	    </collision>
+	    <visual>
+	      <origin xyz="0 0 0.025" rpy="0 0 0"/>
+	      <geometry>
+		<box size="0.05 0.05 0.05"/>
+	      </geometry>
+	      <material name="red">
+		<color rgba="1 0 0 1"/>
+	      </material>
+	    </visual>
+	    <inertial>
+	      <mass value="1e-5" />
+	      <origin xyz="0 0 0" rpy="0 0 0"/>
+	      <inertia ixx="1e-6" ixy="0" ixz="0" iyy="1e-6" iyz="0" izz="1e-6" />
+	    </inertial>
+  </link>
+  <joint name="camera_joint" type="fixed">
+	    <axis xyz="0 1 0" />
+	    <origin xyz="0 0 0.05" rpy="0 0 0"/>
+	    <parent link="arm_link_04"/>
+	    <child link="camera_link"/>
+	 </joint>
 <link name="right_grip_link">
   	<inertial>

File: erl2/urdf/robot.urdf (robot description, URDF)
Before this commit: robot m2wr, 12 links, 11 joints
Links:
- added link camera_link, mass 1e-5; collision box size=0.05 0.05 0.05; visual box size=0.05 0.05 0.05
Joints:
- added joint camera_joint: type fixed, parent cluedo_link, child camera_link, origin xyz=0 0 0.05 rpy=0 0 0, axis 0 1 0
- joint arm_joint_02: limit lower=-1.7 upper=-0.19 effort=1000.0 velocity=0.2 -> lower=-3.14 upper=3.14 effort=1000.0 velocity=0.2
- joint arm_joint_03: limit lower=-1.8 upper=-0.28 effort=1000.0 velocity=0.2 -> lower=-3.14 upper=3.14 effort=1000.0 velocity=0.2
- joint cluedo_joint: axis 1 0 0 -> 0 0 0

Commit message: gmapping imporvements

File: erl2/urdf/m2wr_arm2.xacro (robot description, xacro)
@@ -4,5 +4,5 @@
  <xacro:include filename="$(find erl2)/urdf/m2wr_arm2.gazebo" />
  <!--Define coeff to change proportionally the length of the arm-->
- <xacro:property name="len_coeff" value="0.8" />
+ <xacro:property name="len_coeff" value="0.6" />
  <xacro:macro name="cylinder_inertia" params="mass r l">
     <inertia ixx="${mass*(3*r*r+l*l)/12}" ixy = "0" ixz = "0"

File: erl2/urdf/robot.urdf (robot description, URDF)
Before this commit: robot m2wr, 13 links, 12 joints
Links:
- link arm_link_01: geometry collision cylinder length=0.6 radius=0.04; visual cylinder length=0.6 radius=0.04
- link arm_link_02: geometry collision cylinder length=0.6 radius=0.04; visual cylinder length=0.6 radius=0.04
- link arm_link_03: geometry collision cylinder length=0.6 radius=0.04; visual cylinder length=0.6 radius=0.04
Joints:
- joint arm_joint_01: origin xyz=0 0 0.4 rpy=0 0 0 -> xyz=0 0 0.3 rpy=0 0 0
- joint arm_joint_02: origin xyz=0 0 0.4 rpy=0 0 0 -> xyz=0 0 0.3 rpy=0 0 0
- joint arm_joint_03: origin xyz=0 0 0.8 rpy=0 0 0 -> xyz=0 0 0.6 rpy=0 0 0
- joint arm_joint_04: origin xyz=0 0 0.8 rpy=0 0 0 -> xyz=0 0 0.6 rpy=0 0 0
- joint camera_joint: parent cluedo_link -> arm_link_04

Commit message: removed cluedo_link

File: erl2/urdf/m2wr_arm2.xacro (robot description, xacro)
@@ -248,29 +248,7 @@
   	<child link="arm_link_04"/>
   </joint>
-    <link name="cluedo_link">
-  	<collision>
-  	  <origin xyz="0 0 ${len_coeff*0}" rpy="0 0 1.57"/>
-      <geometry>
-        <box size="0.0001 0.0001 0.0001"/>
-      </geometry>
-  	</collision>
-  	<visual>
-  	  <origin xyz="0 0 ${len_coeff*0}" rpy="0 0 1.57"/>
-      <geometry>
-        <box size="0.0001 0.0001 0.0001"/>
-      </geometry>
-      <material name="red" />
-  	</visual>
-  </link>
-    <joint name="cluedo_joint" type="revolute">
-  	<axis xyz="0 0 0"/>
-  	<limit effort="1000.0" lower="-1.8" upper="1.8" velocity="0.5"/>
-  	<origin rpy="0 0 0" xyz="0 0 0"/>
-  	<parent link="arm_link_04"/>
-  	<child link="cluedo_link"/>
-  </joint>
   <link name="camera_link">
 	    <collision>
-	      <origin xyz="0 0 0.025" rpy="0 0 0"/>
+	      <origin xyz="0 0 0.025" rpy="0 0 1.57"/>
 	      <geometry>
 		<box size="0.05 0.05 0.05"/>
@@ -392,14 +370,4 @@
 	</actuator>
 </transmission>
-<transmission name="cluedo_joint_trans">
-	<type>transmission_interface/SimpleTransmission</type>
-	<joint name="cluedo_joint">
-		<hardwareInterface>hardware_interface/EffortJointInterface</hardwareInterface>
-	</joint>
-	<actuator name="motor5">
-		<hardwareInterface>hardware_interface/EffortJointInterface</hardwareInterface>
-		<mechanicalInterface>1</mechanicalInterface>
-	</actuator>
-</transmission>
 <transmission name="left_grip_trans">
 	<type>transmission_interface/SimpleTransmission</type>

File: erl2/urdf/robot.urdf (robot description, URDF)
Before this commit: robot m2wr, 13 links, 12 joints
Links:
- removed link cluedo_link
Joints:
- removed joint cluedo_joint

Commit message: Bug in init_arm() in movearm.cpp

File: erl2/urdf/m2wr_arm2.xacro (robot description, xacro)
@@ -250,5 +250,5 @@
   <link name="camera_link">
 	    <collision>
-	      <origin xyz="0 0 0.025" rpy="0 0 1.57"/>
+	      <origin xyz="0 0 0.025" rpy="0 0 0"/>
 	      <geometry>
 		<box size="0.05 0.05 0.05"/>
@@ -266,5 +266,5 @@
 	    <inertial>
 	      <mass value="1e-5" />
-	      <origin xyz="0 0 0" rpy="0 0 0"/>
+	      <origin xyz="0 0 0.25" rpy="0 0 0"/>
 	      <inertia ixx="1e-6" ixy="0" ixz="0" iyy="1e-6" iyz="0" izz="1e-6" />
 	    </inertial>
@@ -272,5 +272,5 @@
   <joint name="camera_joint" type="fixed">
 	    <axis xyz="0 1 0" />
-	    <origin xyz="0 0 0.05" rpy="0 0 0"/>
+	    <origin xyz="0 0 0.05" rpy="0 0 1.57"/>
 	    <parent link="arm_link_04"/>
 	    <child link="camera_link"/>

File: erl2/urdf/robot.urdf (robot description, URDF)
Before this commit: robot m2wr, 12 links, 11 joints
Joints:
- joint camera_joint: origin xyz=0 0 0.05 rpy=0 0 0 -> xyz=0 0 0.05 rpy=0 0 1.57

Commit message: fix ontology interface node and progress in state machine

File: erl2/urdf/m2wr_arm2.xacro (robot description, xacro)
@@ -283,13 +283,13 @@
   	</inertial>
   	<collision>
-  	  <origin xyz="-0.032 0.048 0.04" rpy="0 3.1415 -1.57"/>
-      <geometry>
-        <box size="0.06 0.02 0.08"/>
-      </geometry>
-  	</collision>
-  	<visual>
-  	  <origin xyz="-0.032 0.048 0.04" rpy="0 3.1415 -1.57"/>
-      <geometry>
-        <box size="0.06 0.02 0.08"/>
+  	  <origin xyz="-0.032 0.048 0.01" rpy="0 3.1415 -1.57"/>
+      <geometry>
+        <box size="0.06 0.02 0.04"/>
+      </geometry>
+  	</collision>
+  	<visual>
+  	  <origin xyz="-0.032 0.048 0.01" rpy="0 3.1415 -1.57"/>
+      <geometry>
+        <box size="0.06 0.02 0.04"/>
       </geometry>
       <material name="white" />
@@ -298,5 +298,5 @@
   <joint name="right_grip_joint" type="prismatic">
   	<axis xyz="1 0 0"/>
-  	<limit effort="1000.0" lower="-0.04" upper="0.035" velocity="6.5"/>
+  	<limit effort="1000.0" lower="-0.01" upper="0.035" velocity="6.5"/>
   	<origin rpy="0 0 0" xyz="-0.015 0 0.0"/>
   	<parent link="arm_link_04"/>
@@ -310,13 +310,13 @@
   	</inertial>
   	<collision>
-  	  <origin xyz="0.06 0.048 0.04" rpy="0 3.1415 -1.57"/>
-      <geometry>
-        <box size="0.06 0.02 0.08"/>
-      </geometry>
-  	</collision>
-  	<visual>
-  	  <origin xyz="0.06 0.048 0.04" rpy="0 3.1415 -1.57"/>
-      <geometry>
-        <box size="0.06 0.02 0.08"/>
+  	  <origin xyz="0.06 0.048 0.01" rpy="0 3.1415 -1.57"/>
+      <geometry>
+        <box size="0.06 0.02 0.04"/>
+      </geometry>
+  	</collision>
+  	<visual>
+  	  <origin xyz="0.06 0.048 0.01" rpy="0 3.1415 -1.57"/>
+      <geometry>
+        <box size="0.06 0.02 0.04"/>
       </geometry>
       <material name="white" />
@@ -325,5 +325,5 @@
   <joint name="left_grip_joint" type="prismatic">
   	<axis xyz="1 0 0"/>
-  	<limit effort="1000.0" upper="0.04" lower="-0.035" velocity="6.5"/>
+  	<limit effort="1000.0" upper="0.01" lower="-0.035" velocity="6.5"/>
   	<origin rpy="0 0 0" xyz="-0.015 0 0.0"/>
   	<parent link="arm_link_04"/>

File: erl2/urdf/robot.urdf (robot description, URDF)
Before this commit: robot m2wr, 12 links, 11 joints
Links:
- link left_grip_link: geometry collision box size=0.06 0.02 0.04; visual box size=0.06 0.02 0.04
- link right_grip_link: geometry collision box size=0.06 0.02 0.04; visual box size=0.06 0.02 0.04
Joints:
- joint left_grip_joint: limit lower=-0.035 upper=0.04 effort=1000.0 velocity=6.5 -> lower=-0.035 upper=0.01 effort=1000.0 velocity=6.5
- joint right_grip_joint: limit lower=-0.04 upper=0.035 effort=1000.0 velocity=6.5 -> lower=-0.01 upper=0.035 effort=1000.0 velocity=6.5

Commit message: upload stuff and move to docker

File: erl2/urdf/m2wr_arm2.xacro (robot description, xacro)
@@ -276,58 +276,4 @@
 	    <child link="camera_link"/>
 	 </joint>
-<link name="right_grip_link">
-  	<inertial>
-  		<mass value="0.01"/>
-  		<origin xyz="0 0 0" rpy="0 0 0" />
-  		<inertia ixx="0.000010279" ixy="0" ixz="0" iyy="0.000010279" iyz="0" izz="0.000007225"/>
-  	</inertial>
-  	<collision>
-  	  <origin xyz="-0.032 0.048 0.01" rpy="0 3.1415 -1.57"/>
-      <geometry>
-        <box size="0.06 0.02 0.04"/>
-      </geometry>
-  	</collision>
-  	<visual>
-  	  <origin xyz="-0.032 0.048 0.01" rpy="0 3.1415 -1.57"/>
-      <geometry>
-        <box size="0.06 0.02 0.04"/>
-      </geometry>
-      <material name="white" />
-  	</visual>
-  </link>
-  <joint name="right_grip_joint" type="prismatic">
-  	<axis xyz="1 0 0"/>
-  	<limit effort="1000.0" lower="-0.01" upper="0.035" velocity="6.5"/>
-  	<origin rpy="0 0 0" xyz="-0.015 0 0.0"/>
-  	<parent link="arm_link_04"/>
-  	<child link="right_grip_link"/>
-  </joint>
-  <link name="left_grip_link">
-  	<inertial>
-  		<mass value="0.01"/>
-  		<origin xyz="0 0 0" rpy="0 0 0" />
-  		<inertia ixx="0.000010279" ixy="0" ixz="0" iyy="0.000010279" iyz="0" izz="0.000007225"/>
-  	</inertial>
-  	<collision>
-  	  <origin xyz="0.06 0.048 0.01" rpy="0 3.1415 -1.57"/>
-      <geometry>
-        <box size="0.06 0.02 0.04"/>
-      </geometry>
-  	</collision>
-  	<visual>
-  	  <origin xyz="0.06 0.048 0.01" rpy="0 3.1415 -1.57"/>
-      <geometry>
-        <box size="0.06 0.02 0.04"/>
-      </geometry>
-      <material name="white" />
-  	</visual>
-  </link>
-  <joint name="left_grip_joint" type="prismatic">
-  	<axis xyz="1 0 0"/>
-  	<limit effort="1000.0" upper="0.01" lower="-0.035" velocity="6.5"/>
-  	<origin rpy="0 0 0" xyz="-0.015 0 0.0"/>
-  	<parent link="arm_link_04"/>
-  	<child link="left_grip_link"/>
-  </joint>
 <transmission name="arm_joint_01_trans">
 	<type>transmission_interface/SimpleTransmission</type>
@@ -370,23 +316,3 @@
 	</actuator>
 </transmission>
-<transmission name="left_grip_trans">
-	<type>transmission_interface/SimpleTransmission</type>
-	<joint name="left_grip_joint">
-		<hardwareInterface>hardware_interface/EffortJointInterface</hardwareInterface>
-	</joint>
-	<actuator name="motor6">
-		<hardwareInterface>hardware_interface/EffortJointInterface</hardwareInterface>
-		<mechanicalInterface>1</mechanicalInterface>
-	</actuator>
-</transmission>
-<transmission name="right_grip_trans">
-	<type>transmission_interface/SimpleTransmission</type>
-	<joint name="right_grip_joint">
-		<hardwareInterface>hardware_interface/EffortJointInterface</hardwareInterface>
-	</joint>
-	<actuator name="motor7">
-		<hardwareInterface>hardware_interface/EffortJointInterface</hardwareInterface>
-		<mechanicalInterface>1</mechanicalInterface>
-	</actuator>
-</transmission>
 </robot>

File: erl2/urdf/robot.urdf (robot description, URDF)
Before this commit: robot m2wr, 12 links, 11 joints
Links:
- removed link left_grip_link
- removed link right_grip_link
Joints:
- removed joint left_grip_joint
- removed joint right_grip_joint
